Commit message: 更改meshes路径

File: models/mjcf/inspire_hand_arm/hand_mjcf/inspire_right_hand.urdf (robot description, URDF)
Before this commit: robot urdf_right_2025_1_17, 16 links, 15 joints
Links:
- link base_link: geometry collision mesh filename=../../../meshes/base_link.STL; visual mesh filename=../../../meshes/base_link.STL
- link palm_Link: geometry collision mesh filename=../../../meshes/palm_Link.STL; visual mesh filename=../../../meshes/palm_Link.STL
- link palm_Link_1: geometry collision mesh filename=../../../meshes/palm_Link_1.STL; visual mesh filename=../../../meshes/palm_Link_1.STL
- link right_index_1: geometry collision mesh filename=../../../meshes/right_index_1.STL; visual mesh filename=../../../meshes/right_index_1.STL
- link right_index_2: geometry collision mesh filename=../../../meshes/right_index_2.STL; visual mesh filename=../../../meshes/right_index_2.STL
- link right_little_1: geometry collision mesh filename=../../../meshes/right_little_1.STL; visual mesh filename=../../../meshes/right_little_1.STL
- link right_little_2: geometry collision mesh filename=../../../meshes/right_little_2.STL; visual mesh filename=../../../meshes/right_little_2.STL
- link right_middle: geometry collision mesh filename=../../../meshes/right_middle.STL; visual mesh filename=../../../meshes/right_middle.STL
- link right_middle_2: geometry collision mesh filename=../../../meshes/right_middle_2.STL; visual mesh filename=../../../meshes/right_middle_2.STL
- link right_ring_1: geometry collision mesh filename=../../../meshes/right_ring_1.STL; visual mesh filename=../../../meshes/right_ring_1.STL
- link right_ring_2: geometry collision mesh filename=../../../meshes/right_ring_2.STL; visual mesh filename=../../../meshes/right_ring_2.STL
- link right_thumb_1: geometry collision mesh filename=../../../meshes/right_thumb_1.STL; visual mesh filename=../../../meshes/right_thumb_1.STL
- link right_thumb_2: geometry collision mesh filename=../../../meshes/right_thumb_2.STL; visual mesh filename=../../../meshes/right_thumb_2.STL
- link right_thumb_3: geometry collision mesh filename=../../../meshes/right_thumb_3.STL; visual mesh filename=../../../meshes/right_thumb_3.STL
- link right_thumb_4: geometry collision mesh filename=../../../meshes/right_thumb_4.STL; visual mesh filename=../../../meshes/right_thumb_4.STL
